File: kicad/outputs.kicad_sch (KiCad schematic)
At the start: 121 parts, among them J501 OUT 1-8, J502 OUT 9-16, Q501 DMN6075S, Q502 DMN6075S, Q503 DMN6075S, Q504 DMN6075S, Q505 DMN6075S, Q506 DMN6075S, Q507 DMN6075S, Q508 DMN6075S, Q509 DMN6075S, Q510 DMN6075S, Q511 DMN6075S, Q512 DMN6075S, Q513 DMN6075S, Q514 DMN6075S, Q515 DMN6075S, Q516 DMN6075S, U501 TLP291-4, U502 TLP291-4, U503 TLP291-4, U504 TLP291-4

Commit message: - bỏ các mạch 0-10v, RS485 RTU
Parts:
- removed U501, U502, U503, U504: TLP291-4, Package_SO:SOIC-16_4.55x10.3mm_P1.27mm, symbol Isolator:TLP291-4
- added U501, U502, U503, U504, U505, U506, U507, U508, U509, U510, U511, U512, U513, U514, U515, U516: PC817 (SMD), Package_DIP:SMDIP-4_W9.53mm, symbol Isolator:PC817
Connections:
- net GND: now also U501.2, U502.2, U503.2, U504.2, U505.2, U506.2, U507.2, U508.2, U509.2, U510.2, U511.2, U512.2, U513.2, U514.2, U515.2, U516.2
- net at R501.2: now also U501.1
- net at Q509.1 (G), R535.1: now also U509.3
- net at R562.2: now also U516.4
- net at Q502.1 (G), R507.1: now also U502.3
- net at R534.2: now also U509.4
- net at Q516.1 (G), R563.1: now also U516.3
- net at Q513.1 (G), R551.1: now also U513.3
- net at Q510.1 (G), R539.1: now also U510.3
- net at R538.2: now also U510.4
- net at R537.2: now also U510.1
- net at Q512.1 (G), R547.1: now also U512.3
- net at R525.2: now also U507.1
- net at R521.2: now also U506.1
- net at Q504.1 (G), R515.1: now also U504.3
- net at R541.2: now also U511.1
- net at R542.2: now also U511.4
- net at Q511.1 (G), R543.1: now also U511.3
- net at R517.2: now also U505.1
- net at R506.2: now also U502.4
- net at R505.2: now also U502.1
- net at R514.2: now also U504.4
- net at R513.2: now also U504.1
- net at Q507.1 (G), R527.1: now also U507.3
- net at R561.2: now also U516.1
- net at Q508.1 (G), R531.1: now also U508.3
- net at Q503.1 (G), R511.1: now also U503.3
- net at Q501.1 (G), R503.1: now also U501.3
- net at Q515.1 (G), R559.1: now also U515.3
- net at R546.2: now also U512.4
- net at Q514.1 (G), R555.1: now also U514.3
- net at R526.2: now also U507.4
- net at Q506.1 (G), R523.1: now also U506.3
- net at R509.2: now also U503.1
- net at R557.2: now also U515.1
- net at R554.2: now also U514.4
- net at R553.2: now also U514.1
- net at R558.2: now also U515.4
- net at R533.2: now also U509.1
- net at R549.2: now also U513.1
- net at R550.2: now also U513.4
- net at R522.2: now also U506.4
- net at R510.2: now also U503.4
- net at R518.2: now also U505.4
- net at R529.2: now also U508.1
- net at Q505.1 (G), R519.1: now also U505.3
- net at R530.2: now also U508.4
- net at R502.2: now also U501.4
- net at R545.2: now also U512.1
Other:
- note added: "16 NGO RA TRANSISTOR SINK (NPN-type): MCU -> PC817 -> MOSFET 60V/2.5A. Tai noi giua V+ (24V) va Yn. Cap nguon ngoai vao V+/COM (cach ly voi mach logic)."
- note removed: "16 NGO RA TRANSISTOR SINK (NPN-type): MCU -> TLP291 -> MOSFET 60V/2.5A. Tai noi giua V+ (24V) va Yn. Cap nguon ngoai vao V+/COM (cach ly voi mach logic)."

Commit message: - bỏ các cầu chì thêm mô tả cho từng linh kiên
Other:
- note added: "D533 TVS 33V + C501 10µF/50V + C502 100nF: bảo vệ và lọc nguồn tải V+."
- note added: "DOx = 1 → LED opto sáng → MOSFET dẫn → Yn kéo về COM → relay hút."
- note added: "KÊNH NGÕ RA (16 kênh giống nhau) – SINK, CÁCH LY QUANG"
- note added: "LED Qn: I = (24V − 2V)/10kΩ ≈ 2.2mA – báo trạng thái ngõ ra thực."
- note added: "MOSFET 60V/2.5A, R_on≈0.1Ω: P = 0.5²×0.1 = 25mW (relay 0.5A); tắt τ≈R_g·C_iss≈3µs."
- note added: "Nguồn relay 12–30V vào V+ (chân 2) / COM (chân 1). Tải nối giữa V+ và Yn. KHÔNG nối COM với GND board (mất cách ly). Giới hạn 30V: Vceo PC817 = 35V."
- note added: "PC817: cách ly 5000Vrms; CTR ≥ 50% → I_C ≥ 2.2mA."
- note added: "R_c 10k + R_g 10k: V_GS = V+ × 10k/20k = V+/2 ≈ 12V @24V (V_GS max 20V → V+ ≤ 30V; ≥ 4.5V → V+ ≥ 10V). I_opto = 24V/20k = 1.2mA < 2.2mA → bão hòa."
- note added: "R_in 470Ω: I_F = (3.3V − 1.2V)/470Ω ≈ 4.5mA (PC817 ~5mA; GPIO ≤ 25mA)."
- note added: "SS16: dập xung ngược L·di/dt của cuộn relay về V+."
