File: kicad/usb.kicad_sch (KiCad schematic)
At the start: 20 parts, among them J301 USB-C, Q301 MMBT3904, Q302 MMBT3904, Q303 MMBT3906, U301 USBLC6-2SC6, U302 CH340C

Commit message: - bỏ các cầu chì thêm mô tả cho từng linh kiên
Other:
- note added: "(RTS=1, DTR=0) → reset; (RTS=0, DTR=1) → nhả reset với BOOT0 = 1 → MCU vào bootloader. RTS, DTR cùng mức: không tác động."
- note added: "CH340C – USB ↔ UART (nạp code)"
- note added: "Dao động nội, không cần thạch anh. Cấp 3.3V nên V3 nối VCC. TXD/RXD → USART1 (PA9/PA10) = cổng bootloader ROM của STM32. C303 100nF + C304 10µF lọc nguồn."
- note added: "F301 PTC 500mA: bảo vệ cổng USB máy tính (USB 2.0 ≤ 500mA). C302 1µF lọc VBUS."
- note added: "JP301: bật/tắt nạp tự động. R308 1k hạn dòng khi nút BOOT và mạch tự động cùng tác động (≤ 3.3mA)."
- note added: "Q301: RTS=1, DTR=0 → kéo NRST xuống. I_B = (3.3 − 0.7)/10k ≈ 0.26mA → bão hòa (β ≥ 100)."
- note added: "Q302: RTS=0, DTR=1 → kéo BOOT_N xuống. R306 10k kéo BOOT_N lên khi nghỉ."
- note added: "Q303 (PNP) dẫn khi BOOT_N = 0 → BOOT0 = 3.3V. R307 hạn dòng bazơ."
- note added: "R301, R302 5.1kΩ = R_d chuẩn Type-C: máy tính/sạc nhận ra thiết bị → cấp 5V lên VBUS."
- note added: "TỰ VÀO BOOTLOADER BẰNG DTR/RTS"
- note added: "USBLC6-2SC6: chống ESD ±15kV cho D+, D−, VBUS."
- note added: "Vỏ USB → GND qua 1MΩ // 4.7nF: xả tĩnh điện chậm, nhiễu cao tần qua tụ, tránh vòng đất."
